Commit message: Restructuring

File: Siclo1.urdf (robot description, URDF)
Before this commit: robot Siclo1, 11 links, 10 joints
Joints:
- joint Left_Ankle: origin xyz=0.1 0.024043 -0.679218 rpy=0 0 0 -> xyz=0.0 0.0 -0.686961 rpy=0 0 0
- joint Left_Hip_Twist: origin xyz=0.925 0.2 0.98 rpy=0 0 0 -> xyz=0.925 0.2 1.018094 rpy=0 0 0
- joint Left_Knee: origin xyz=0.031 0.000969 -0.052133 rpy=0 0 0 -> xyz=0.0 0.0 -0.060661 rpy=0 0 0
- joint Right_Hip_Twist: limit lower=-0.034907 upper=0.349066 effort=100 velocity=100 -> lower=-0.349066 upper=0.349066 effort=100 velocity=100
